File: mine/CH634W6G hub/CH634W6G hub.kicad_sch (KiCad schematic)
At the start: 5 parts, among them U1 CH634W6G, U2 *, U3 CH211D

Commit message: got the protection in?
Parts:
- added U4: *, CHXXX:SOT-23-6, symbol CHXXX:CH217K
- R1: value 24k -> 30k
- R2: value 51k -> 30k
Connections:
- net +5V: now also U4.6 (VIN)
- net GND: now also R2.1, U1.0 (GND), U1.16 (GND), U1.18 (GND_DCDC), U4.2 (GND)
- net PWRSTART: now also U4.4 (EN#)
- net PWRSTOP: now also U4.3 (FLAG#); no longer R2.1
- net VBUS: now also U4.1 (VOUT)
- net VDD5: now reaches U1.20 (VDD5)
- net VDD33: now reaches U1.21 (VDD33/VIO33)
- net VDD33: now also U1.35 (AVDD33), U1.54 (VIO33)
- net +3.3V: no longer names the net of R2.2
- net +3.3V: now also U4.5 (ISET)
Other:
- note added: "Current limit=Resistor on Flag#/Resistor on ISet = 60k/30k = 2A Global overcurrent limit for the 4 usb is 4A the usb spec says that a device should draw no more then .9A"
- note added: "usually the overcurrent (PWRSTOP) pin needs to be pulled up, CH634W6G does this"
- note removed: "Current limit=Resistor on Flag#/Resistor on ISet = 51k/24k = 2.125A Global current limit for the 4 usb A"
- moved on the sheet: R1, U1, U2, U3

Commit message: all
Parts:
- added C1, C5: 1uF, fab:C_0603, symbol fab:C_0603
- added C2, C6: 10uF, fab:C_0603, symbol fab:C_0603
- added C3, C4, C7, C8: 0.1uF, fab:C_0603, symbol fab:C_0603
Connections:
- net GND: now also C1.2, C2.2, C3.2, C4.1, C5.2, C6.2, C7.2, C8.2
- net VDD33: now also C1.1, C2.1, C3.1, C4.2
- net VDD5: now also C5.1, C6.1
- net at U1.17 (VFB): now also C7.1
- net VDD12: now reaches U1.19 (VSW)
- net VDD12: now also U1.27 (DVDD12), C8.1
- net XO: now reaches U1.44 (XO)
- net XI: now reaches U1.45 (XI)
- no-connect marks 0 -> 7

Commit message: got a bit more pins labeled
Parts:
- removed C1, C5: 1uF, fab:C_0603, symbol fab:C_0603
- removed C2, C6: 10uF, fab:C_0603, symbol fab:C_0603
- removed C3, C4, C7, C8: 0.1uF, fab:C_0603, symbol fab:C_0603
Connections:
- net VFB: now reaches U1.17 (VFB)
- net CFG0: now reaches U1.22 (CFG0)
- net CFG1: now reaches U1.23 (CFG1)
- net VDD33/VIO33: now reaches U1.24 (RESET#)
- net VDD33/VIO33: now also U1.21 (VDD33/VIO33), U1.54 (VIO33)
- net VDD12 renamed DVDD12
- net DVDD12: no longer U1.19 (VSW)
- removed net VDD33: U1.21 (VDD33/VIO33), U1.35 (AVDD33), U1.54 (VIO33)
- new net AVDD33: U1.35 (AVDD33)
- new net VSW: U1.19 (VSW)
- no-connect marks 7 -> 9
Other:
- moved on the sheet: R1, R2, U2, U4

Commit message: why am I even redesigning the schematic, im just gonna use example, this is a backup
Parts:
- added C1, C5: 1uF, fab:C_0603, symbol fab:C_0603
- added C10, C11, C12, C13, C14, C2, C8, C9: 0.1uF, fab:C_0603, symbol fab:C_0603
- added C15, C3: 15pF, fab:C_0603, symbol fab:C_0603
- added C16, C17: 20pF, 0402_C, symbol *:root_0_CAP_*_0
- added C16, C17, C20, C25, C27, C29, C43: 10uF, 0603_C, symbol *:root_0_CAP_*_0
- added C18: NC(0.1uF), 0402_C, symbol *:root_1_CAP_*_0
- added C18, C19, C20, C21, C22, C23, C28, C30: 0.1uF, 0402_C, symbol *:root_2_CAP_*_0
- added C19: 1uF, 0402_C, symbol Miscellaneous Devices:root_1_Cap_Miscellaneous Devices.IntLib
- added C21: 1uF, 0402_C, symbol wch_sch_others:root_1_CAP_wch_sch_others.schLib_0
- added C22: 100nF, 0402_C, symbol wch_sch_others:root_0_CAP_wch_sch_others.schLib_0
- added C23, C24, C25, C26, C27, C30, C32, C33, C34, C35: 0.1uF, 0201_C, symbol *:root_1_CAP_*_0
- added C24: 0.1uF, 0402_C, symbol *:root_0_CAP_*_0
- added C26: 10uF, 0603_C, symbol Miscellaneous Devices:root_1_Cap_Miscellaneous Devices.IntLib
- added C28: 1uF, 0402_C, symbol wch_sch_others:root_1_mirrored_CAP_wch_sch_others.schLib_0
- added C29, C40: 1uF, 0402_C, symbol wch_sch_others:root_3_CAP_wch_sch_others.schLib_0
- added C31: 1uF, 0402_C, symbol *:root_1_CAP_*_0
- added C36: 100nF, 0402_C, symbol Miscellaneous Devices LC:root_2_0603 100nF (104) 10% 50V_Miscellaneous Devices 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
- added C37, C38, C39: 22uF, 0805_C, symbol Miscellaneous Devices LC:root_1_0603 100nF (104) 10% 50V_Miscellaneous Devices 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
- added C4, C6, C7: 10uF, fab:C_0603, symbol fab:C_0603
- added C41: 1uF, 0402_C, symbol Miscellaneous Devices LC:root_1_0603 100nF (104) 10% 50V_Miscellaneous Devices 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
- added C42: 1uF, 0402_C, symbol wch_sch_others:root_2_CAP_wch_sch_others.schLib_0
- added C45: 0.1uF, 0402_C, symbol Miscellaneous Devices:root_1_Cap_Miscellaneous Devices.IntLib
- added D1: SS34, SOD-123, symbol CHXXX:root_0_DIODE_CHXXX.schlib_0
- added D2: SS34, SOD-123, symbol CHXXX:root_0_mirrored_DIODE_CHXXX.schlib_0
- added L1: 2.2uH, Personal:0603, symbol 0603:L_0603
- added L2: 2.2uH, CD32, symbol Miscellaneous Devices:root_0_Inductor_Miscellaneous Devices.IntLib
- added L2: 15uH, IND-SMD_L7.0-W6.6, symbol wch_sch_others:root_0_INDUCTOR_wch_sch_others.schLib
- added LED2: 5V, 0603+, symbol *:root_3_LED_*_0
- added P1: PORT1, USB-3.0F-TL, symbol *:root_0_USB-AF3.0-90卷_*_0
- added P2: PORT2, USB-3.0F-TL, symbol *:root_0_USB-AF3.0-90卷_*_0
- added P3: PORT3, USB-3.0F-TL, symbol *:root_0_USB-AF3.0-90卷_*_0
- added P4: PORT4, USB-3.0F-TL, symbol *:root_0_USB-AF3.0-90卷_*_0
- added P5: UP, CABLE-TYPEC1, symbol wch_sch_others:root_0_TypeC-Cable1_wch_sch_others.schLib
- added P6: TYPE-C, TYPE-C-Receptacle-2.0-16PIN-L6.5mmSinkDown1.2mm, symbol wch_sch_others:root_3_TYPE-C-1_wch_sch_others.schLib_0
- added P7: (no value), SIP3-2.54mm, symbol Miscellaneous Connectors:root_2_Header 3_Miscellaneous Connectors.IntLib
- added P8: (no value), SIP5-2.54mm, symbol wch_sch_others:root_2_HEADER 5_wch_sch_others.schLib_0
- added Q1: SE3060D, DFN-8_L3.1-W3.0-P0.65-LS3.3-BL, symbol wch_sch_others:root_1_mirrored_N-MOS 8pin_wch_sch_others.schLib
- added Q2: SE3060D, DFN-8_L3.1-W3.0-P0.65-LS3.3-BL, symbol wch_sch_others:root_1_N-MOS 8pin_wch_sch_others.schLib
- added R10, R13: NC(51K), 0402, symbol *:root_3_RES_*_0
- added R11, R8: 24K, 0402, symbol *:root_1_RES_*_0
- added R12: NC(10K), 0402, symbol *:root_1_mirrored_RES_*_0
- added R14: 0Ω(10K), 0402, symbol *:root_1_RES_*_0
- added R15: 5.1KΩ, 0402, symbol Miscellaneous Devices LC:root_0_0603 56KΩ (5602) 1%_Miscellaneous Devices LC.In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
- added R18, R19, R3: 10K, 0402, symbol *:root_1_RES_*_0
- added R20, R21, R9: NC(10K), 0402, symbol *:root_1_RES_*_0
- added R24: 105K, 0402, symbol wch_sch_others(1):root_1_RES_wch_sch_others(1).SchLib_0
- added R25: 20K, 0402, symbol wch_sch_others(1):root_1_RES_wch_sch_others(1).SchLib_0
- added R3, R4: 10K, 0402, symbol Miscellaneous Devices LC:root_3_0603 56KΩ (5602) 1%_Miscellaneous Devices LC.In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
- added R4, R5: 680KΩ, 0402, symbol Miscellaneous Devices LC:root_3_0603 56KΩ (5602) 1%_Miscellaneous Devices LC.In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
- added R6: 1KΩ, 0402, symbol Miscellaneous Devices LC:root_3_0603 56KΩ (5602) 1%_Miscellaneous Devices LC.In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
- added R7: 2K, 0402, symbol *:root_1_RES_*_0
- added TP1, TP2: Testpoint, TESTPOINT3, symbol wch_sch_others:root_3_Testpoint_wch_sch_others.schLib
- added U5: CH634W6G, QFN64_8X8, symbol CHXXX:root_0_CH634W6G_CHXXX.schlib
- added U6: CH211C, QFN16C_2X2, symbol CHXXX:root_0_CH211C_CHXXX.schlib_0
- added U6: ETA2807, SOT-23-6, symbol wch_sch_others:root_0_TPS54202_wch_sch_others.schLib
- added U7, U8: CH217K, SOT-23-6, symbol CHXXX:root_0_CH217K_CHXXX.schlib
- added X1: TAXM24M4ZDBCCT2T, EasyEDA:CRYSTAL-SMD_4P-L2.0-W1.6-BL-A, symbol EasyEDA:TAXM24M4ZDBCCT2T
- added X2: 24MHz, XT3225, symbol *:root_0_晶体_*_0
Connections:
- net DVDD12 is gone; now on net 1V2_HUB: U1.27 (DVDD12)
- net VFB is gone; now on net 1V2_HUB: U1.17 (VFB)
- net AVDD33: now also U1.21 (VDD33/VIO33), U1.54 (VIO33), C1.1, C14.1, C2.1, C24.1, C27.1, C28.2, C30.2, C4.1, C42.1, C43.1, P8.4, R10.1, R13.1, R14.2, R18.2, R19.2, R9.2, U5.21 (VDD33/VIO33), U5.35 (AVDD33), U5.54 (VIO33), U6.1 (VDD33)
- net CFG0: now also R18.1, R20.2, U5.22 (CFG0)
- net CFG1: now also R19.1, R21.2, U5.23 (CFG1)
- net GND: now also C1.2, C10.2, C11.2, C12.2, C13.2, C14.2, C15.2, C16.2, C16.2, C17.1, C17.2, C18.1, C18.1, C19.1, C19.1, C2.2, C20.1, C20.2, C21.1, C21.1, C22.1, C22.1, C23.1, C24.2, C25.2, C26.1, C27.2, C28.1, C28.1, C29.2, C29.2, C3.1, C30.1, C31.1, C37.1, C38.1, C39.1, C4.2, C40.2, C41.1, C42.2, C43.2, C45.1, C5.2, C6.2, C7.2, C8.2, C9.2, LED2.2 (K), P1.0 (EGND), P1.4 (GND), P1.7 (GND), P2.0 (EGND), P2.4 (GND), P2.7 (GND), P3.0 (EGND), P3.4 (GND), P3.7 (GND), P4.0 (EGND), P4.4 (GND), P4.7 (GND), P5.16 (GND), P6.A1 (GND), P6.B1 (GND), P7.3, P8.3, R11.2, R12.1, R15.2, R20.1, R21.1, R25.1, R3.1, R3.2, R4.2, R6.2, R8.2, U5.0 (GND), U5.16 (GND), U5.18 (GND_DCDC), U6.1 (GND), U6.3 (GND), U7.2 (GND), U8.2 (GND), X1.2 (GND), X1.4 (GND), X2.2 (GND), X2.4 (GND)
- net VBUS: now also C21.2, C29.1, D1.1 (A), P5.9 (VCC), Q1.1 (S), Q1.2 (S), Q1.3 (S), R4.1, TP1.1, U6.14 (VBUS)
- net VDD5: now also C26.2, C31.2, C38.2, C39.2, C5.1, C6.1, L2.2, P8.5, R24.2, R7.2, U5.20 (VDD5), U7.6 (VIN), U8.6 (VIN)
- net VSW: now also L1.1, L2.1, U5.19 (VSW)
- net XI: now also C16.1, C3.2, U5.45 (XI), X1.1 (OSC1), X2.1 (XIN)
- net XO: now also C15.1, C17.2, U5.44 (XO), X1.3 (OSC2), X2.3 (XOUT)
- net 1V2_HUB: now reaches U1.13 (P2_VDD12)
- net 1V2_HUB: now also U1.3 (P3_VDD12), U1.40 (UP_VDD12), U1.58 (P4_VDD12), C10.1, C11.1, C12.1, C13.1, C18.2, C19.2, C19.2, C20.1, C20.2, C21.2, C22.2, C23.2, C45.2, C7.1, C8.1, C9.1, L1.2, L2.2, U5.13 (P2_VDD12), U5.17 (VFB), U5.27 (DVDD12), U5.3 (P3_VDD12), U5.40 (UP_VDD12), U5.49 (P1_VDD12), U5.58 (P4_VDD12)
- removed net VDD33/VIO33: U1.21 (VDD33/VIO33), U1.24 (RESET#), U1.54 (VIO33)
- new net: R11.1, U8.5 (ISET)
- new net: C40.1, U6.16 (VDD49)
- new net: C32.1, P3.8 (TX-)
- new net: LED2.1 (A), R7.1
- new net: R24.1, R25.2, U6.4 (FB)
- new net: C30.2, P5.7 (B11)
- new net: C26.1, P2.8 (TX-)
- new net: P5.10 (B5), R6.1
- new net: C41.2, U6.5 (VLDO)
- new net: R8.1, U7.5 (ISET)
- new net: C34.1, P3.9 (TX+)
- new net: C33.1, P4.8 (TX-)
- new net: C27.1, P2.9 (TX+)
- new net: C35.1, P4.9 (TX+)
- new net: C24.1, P1.9 (TX+)
- new net: C25.2, P5.8 (B10)
- new net: C36.1, L2.1, U6.2 (SW)
- new net: C36.2, U6.6 (BST)
- new net: C23.1, P1.8 (TX-)
- new net CC1_P1: P6.A5 (CC1), R15.1, U6.12 (ODH1)
- new net CC1_P2: P5.11 (A5), U6.9 (CCH2)
- new net CC2_P1: P6.B5 (CC2), U6.10 (CCH1)
- new net HVCP: C22.2, R4.2, R5.2, U6.13 (HVCP)
- new net OVCUR#: R10.2, R13.2, U5.33 (OVCUR#), U7.3 (FLAG#), U8.3 (FLAG#)
- new net P1_HS_DM: P1.2 (D-), U5.53 (P1_HS_DM)
- new net P1_HS_DP: P1.3 (D+), U5.52 (P1_HS_DP)
- new net P1_SS_RXA: P1.5 (RX-), U5.51 (P1_SS_RXA)
- new net P1_SS_RXB: P1.6 (RX+), U5.50 (P1_SS_RXB)
- new net P1_SS_TXA: C23.2, U5.48 (P1_SS_TXA)
- new net P1_SS_TXB: C24.2, U5.47 (P1_SS_TXB)
- new net P2_HS_DM: P2.2 (D-), U5.10 (P2_HS_DM)
- new net P2_HS_DP: P2.3 (D+), U5.9 (P2_HS_DP)
- new net P2_SS_RXA: P2.5 (RX-), U5.15 (P2_SS_RXA)
- new net P2_SS_RXB: P2.6 (RX+), U5.14 (P2_SS_RXB)
- new net P2_SS_TXA: C26.2, U5.12 (P2_SS_TXA)
- new net P2_SS_TXB: C27.2, U5.11 (P2_SS_TXB)
- new net P3_HS_DM: P3.2 (D-), U5.7 (P3_HS_DM)
- new net P3_HS_DP: P3.3 (D+), U5.6 (P3_HS_DP)
- new net P3_SS_RXA: P3.5 (RX-), U5.5 (P3_SS_RXA)
- new net P3_SS_RXB: P3.6 (RX+), U5.4 (P3_SS_RXB)
- new net P3_SS_TXA: C32.2, U5.2 (P3_SS_TXA)
- new net P3_SS_TXB: C34.2, U5.1 (P3_SS_TXB)
- new net P4_HS_DM: P4.2 (D-), U5.64 (P4_HS_DM)
- new net P4_HS_DP: P4.3 (D+), U5.63 (P4_HS_DP)
- new net P4_SS_RXA: P4.5 (RX-), U5.60 (P4_SS_RXA)
- new net P4_SS_RXB: P4.6 (RX+), U5.59 (P4_SS_RXB)
- new net P4_SS_TXA: C33.2, U5.57 (P4_SS_TXA)
- new net P4_SS_TXB: C35.2, U5.56 (P4_SS_TXB)
- new net PDHUB#: R3.2, U5.31 (SPI_SCS)
- new net PWREN#: U5.34 (PWREN#), U7.4 (EN#), U8.4 (EN#)
- new net RESET#: C18.2, R14.1, U1.24 (RESET#), U5.24 (RESET#)
- new net RSVD/HUB_CC: P7.2, U5.26 (RSVD/HUB_CC), U6.7 (CCL2)
- new net SPI_MISO/SDA: P8.2, U5.30 (SPI_MISO/SDA), U6.2 (SDA)
- new net SPI_MOSI: U5.28 (SPI_MOSI)
- new net SPI_SCK/SCL: P8.1, U5.29 (SPI_SCK/SCL), U6.4 (SCL)
- new net SUSP/CFG2: R12.2, R9.1, U5.32 (LED/CFG2)
- new net UP_HS_DM: P5.14 (A7), U5.36 (UP_HS_DM)
- new net UP_HS_DP: P5.15 (A6), U5.37 (UP_HS_DP)
- new net UP_SS_RXA: P5.5 (A2), U5.42 (UP_SS_RXA)
- new net UP_SS_RXB: P5.6 (A3), U5.41 (UP_SS_RXB)
- new net UP_SS_TXA: C30.1, U5.39 (UP_SS_TXA)
- new net UP_SS_TXB: C25.1, U5.38 (UP_SS_TXB)
- new net VBUS_DET/PWR_CC: P7.1, U5.25 (VBUS_DET/PWR_CC), U6.6 (CCL1)
- new net VBUS_EN: Q1.4 (G), R4.1, U6.8 (HVIO)
- new net VBUS_OUT: C16.1, C17.1, C25.1, C29.1, P1.1 (VBUS), P2.1 (VBUS), P3.1 (VBUS), P4.1 (VBUS), U7.1 (VOUT), U8.1 (VOUT)
- new net VHV: C37.2, D1.2 (K), D2.2 (K), Q1.5 (D), Q1.6 (D), Q1.7 (D), Q1.8 (D), Q2.5 (D), Q2.6 (D), Q2.7 (D), Q2.8 (D), U6.3 (VIN)
- new net VIN: C28.2, D2.1 (A), P6.A4 (VBUS), P6.B4 (VBUS), Q2.1 (S), Q2.2 (S), Q2.3 (S), R3.1, TP2.1, U6.15 (VSYS)
- new net VIN_EN: Q2.4 (G), R5.1, U6.11 (ODH2)
Other:
- note added: "BC Disable"
- note added: "BC Enable"
- note added: "Configured for a single 5v input"
- note added: "Near pin 20"
- note added: "Near pin 21"
- note added: "Near pin 35"
- note added: "Near pin 3、13、27、40、49、58"
- note added: "Near pin 54"
- note added: "PD MODE"
- note added: "test point"
